File: test/B7Test/B7Test.kicad_pcb (KiCad board)
At the start: 2 copper layers, 0 parts

Commit message: aktueller Stand
Parts:
- added U1: CPDT6-5V0UPC-HF, B7_Footprints:SOT-23-6, F.Cu at (102.5, 82.9)

Commit message: B7 libs, test project
Parts:
- added U2: NE555DR, B7_Footprints:SOIC-8_3.9x4.9mm_P1.27mm, F.Cu at (128.5, 95.0)
- added U3: STM32F446VETx, B7_Footprints:LQFP-100_14x14mm_P0.5mm, F.Cu at (122.0, 78.1)
- added U4: PESD5V0U4BW, B7_Footprints:SOT-665, F.Cu at (151.3, 76.4)
