File: test/B7Test/B7Test.kicad_sch (KiCad schematic)
At the start: 0 parts

Commit message: aktueller Stand
Parts:
- added U1: CPDT6-5V0UPC-HF, B7_Footprints:SOT-23-6, symbol B7_PartDB:CPDT6-5V0UPC-HF
Changed lines of the file:
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@@
 	(generator_version "9.0")
 	(paper "A4")
+	(symbol
+		(lib_id "B7_PartDB:CPDT6-5V0UPC-HF")
+		(at 113.03 71.12 0)
+		(unit 1)
+		(exclude_from_sim yes)
+		(in_bom yes)
+		(on_board yes)
+		(dnp no)
+		(property "Reference" "U1"
+			(at 119.38 69.8499 0)
+			(effects
+				(font
+					(size 1.27 1.27)
+				)
+				(justify left)
+			)
+		)
+		(property "Value" "CPDT6-5V0UPC-HF"
+			(at 119.38 72.3899 0)
+			(effects
+				(font
+					(size 1.27 1.27)
+				)
+				(justify left)
+			)
+		)
+		(property "Footprint" "B7_Footprints:SOT-23-6"
+			(at 114.3 69.215 0)
+			(effects
+				(font
+					(size 1.27 1.27)
+				)
+				(hide yes)
+			)
+		)
+		(property "Datasheet" "https://partdb.midnight-worker.de/en/part/7/info"
+			(at 114.3 69.215 0)
+			(effects
+				(font
+					(size 1.27 1.27)
+				)
+				(hide yes)
+			)
+		)
+		(property "Description" "10A@8/20us 12.5V 125W 6V Unidirectional 5V SOT-23-6 ESD and Surge Protection (TVS/ESD) ROHS"
+			(at 113.03 71.12 0)
+			(effects
+				(font
+					(size 1.27 1.27)
+				)
+				(hide yes)
+			)
+		)
+		(property "Category" "Circuit Protection/ESD and Surge Protection (TVS â ESD)"
+			(at 113.03 71.12 0)
+			(effects
+				(font
+					(size 1.27 1.27)
+				)
+				(hide yes)
+			)
+		)
+		(property "Manufacturer" "Comchip"
+			(at 113.03 71.12 0)
+			(effects
+				(font
+					(size 1.27 1.27)
+				)
+				(hide yes)
+			)
+		)
+		(property "MPN" "CPDT6-5V0UPC-HF"
+			(at 113.03 71.12 0)
+			(effects
+				(font
+					(size 1.27 1.27)
+				)
+				(hide yes)
+			)
+		)
+		(property "Manufacturing Status" ""
+			(at 113.03 71.12 0)
+			(effects
+				(font
+					(size 1.27 1.27)
+				)
+				(hide yes)
+			)
+		)
+		(property "Part-DB Footprint" "SOT-23-6"
+			(at 113.03 71.12 0)
+			(effects
+				(font
+					(size 1.27 1.27)
+				)
+				(hide yes)
+			)
+		)
+		(property "Mass" "0.001 g"
+			(at 113.03 71.12 0)
+			(effects
+				(font
+					(size 1.27 1.27)
+				)
+				(hide yes)
+			)
+		)
+		(property "Part-DB ID" "7"
+			(at 113.03 71.12 0)
+			(effects
+				(font
+					(size 1.27 1.27)
+				)
+				(hide yes)
+			)
+		)
+		(property "Part-DB IPN" "C2443674"
+			(at 124.46 74.676 0)
+			(effects
+				(font
+					(size 1.27 1.27)
+				)
+			)
+		)
+		(pin "6"
+		)
+		(pin "1"
+		)
+		(pin "5"
+		)
+		(pin "2"
+		)
+		(pin "4"
+		)
+		(pin "3"
+		)
+		(instances
+			(project ""
+				(path "/231fd3f6-a7b9-4f74-acca-8f5aa04ca05a"
+					(reference "U1")
+					(unit 1)
+				)
+			)
+		)
+	)
 	(sheet_instances
 		(path "/"

Commit message: B7 libs, test project
Parts:
- added U2: NE555DR, B7_Footprints:SOIC-8_3.9x4.9mm_P1.27mm, symbol B7_PartDB:NE555N-TD
- added U3: STM32F446VETx, B7_Footprints:LQFP-100_14x14mm_P0.5mm, symbol B7_PartDB:STM32F446VET6TR
- added U4: PESD5V0U4BW, B7_Footprints:SOT-665, symbol B7_PartDB:PESD5V0U4BW
Connections:
- new net: U4.2 (A), U4.5 (A)
- new net: U3.10 (VSS), U3.27 (VSS), U3.49 (VSS), U3.74 (VSS), U3.99 (VSS)
